File: PCB/Homeostasis.kicad_sch (KiCad schematic)
At the start: 16 parts, among them J1 USB_A, J2 Conn_02x03_Odd_Even, U2 ATmega328P-P, Y1 16MHz

Commit message: Schematic Update
Parts:
- removed J1: USB_A, symbol Connector:USB_A
- added C10, C11: 100uF, symbol Device:C_Polarized
- added J1: USB_Connector, symbol Connector:Screw_Terminal_01x02
- added J3: Fan_1, symbol Connector_Generic:Conn_01x04
- added J4: Fan_2, symbol Connector_Generic:Conn_01x04
- added Q1, Q2: 2N7002, Package_TO_SOT_SMD:SOT-23, symbol Transistor_FET:2N7002
- added R2, R4: 150, symbol Device:R
- added R3, R5, R6, R7: 10k, symbol Device:R
- C1: value 330uF -> 100uF
- F1: value Polyfuse -> 500mA
- J2: value Conn_02x03_Odd_Even -> ISP_Connector
Connections:
- net GND: now also C10.2, C11.2, J1.2 (Pin_2), J3.1 (Pin_1), J4.1 (Pin_1), Q1.2 (S), Q2.2 (S), R3.1, R5.1
- net at F1.1: now also J1.1 (Pin_1)
- net GATE_1: now reaches U2.15 (PB1)
- net GATE_1: now also R2.2
- net GATE_2: now reaches U2.16 (PB2)
- net GATE_2: now also R4.2
- net TACH_1: now reaches U2.4 (PD2)
- net TACH_1: now also J3.3 (Pin_3), R6.2
- net TACH_2: now reaches U2.5 (PD3)
- net TACH_2: now also J4.3 (Pin_3), R7.2
- net +5V_PROTECTED renamed +5V_P
- net +5V_P: now also C10.1, C11.1, J3.2 (Pin_2), J4.2 (Pin_2), R6.1, R7.1
- new net: Q2.1 (G), R4.1, R5.2
- new net: Q1.1 (G), R2.1, R3.2
- new net PWM_1: J3.4 (Pin_4), Q1.3 (D)
- new net PWM_2: J4.4 (Pin_4), Q2.3 (D)
- no-connect marks 2 -> 0
Other:
- moved on the sheet: C7, F1, R1

Commit message: Schematic Update
Parts:
- added J5: TPROBE_1, symbol Connector_Generic:Conn_01x03
- added J6: TPROBE_2, symbol Connector_Generic:Conn_01x03
- added J7: TPROBE_3, symbol Connector_Generic:Conn_01x03
- added J8: TPROBE_4, symbol Connector_Generic:Conn_01x03
- added J9: OLED, symbol Connector_Generic:Conn_01x04
- added R10, R9: 4.7k DNP, symbol Device:R
- added R11: 4.7k, symbol Device:R
- added R8: 100, symbol Device:R
- added SW1, SW2, SW3, SW4: SW_Push, symbol Switch:SW_Push
- C10, C11: value 100uF -> 47uF
Connections:
- net +5V_P: now also J5.3 (Pin_3), J6.3 (Pin_3), J7.3 (Pin_3), J8.3 (Pin_3), J9.2 (Pin_2), R10.1, R11.2, R9.1
- net GND: now also J5.1 (Pin_1), J6.1 (Pin_1), J7.1 (Pin_1), J8.1 (Pin_1), J9.1 (Pin_1), SW1.2, SW2.2, SW3.2, SW4.2
- net RESET: now also SW4.1
- net SUP: now reaches U2.23 (PC0)
- net SUP: now also SW1.1
- net SDOWN: now reaches U2.24 (PC1)
- net SDOWN: now also SW2.1
- net TUPDATE: now reaches U2.25 (PC2)
- net TUPDATE: now also SW3.1
- net OLED_SDA: now reaches U2.27 (PC4)
- net OLED_SDA: now also J9.4 (Pin_4), R9.2
- net OLED_SCL: now reaches U2.28 (PC5)
- net OLED_SCL: now also J9.3 (Pin_3), R10.2
- net at U2.6 (PD4): now also R8.1
- new net TDATA: J5.2 (Pin_2), J6.2 (Pin_2), J7.2 (Pin_2), J8.2 (Pin_2), R11.1, R8.2
- no-connect marks 0 -> 7
Other:
- moved on the sheet: C9

Commit message: Schematic Update
Parts:
- added H1, H2, H3: MountingHole, MountingHole:MountingHole_3.2mm_M3, symbol Mechanical:MountingHole
- C1: footprint (none) -> Capacitor_THT:CP_Radial_D6.3mm_P2.50mm
- C10, C11: footprint (none) -> Capacitor_THT:CP_Radial_D5.0mm_P2.00mm
- C2: footprint (none) -> Capacitor_SMD:C_1206_3216Metric
- C3, C4, C5, C6, C7, C8: footprint (none) -> Capacitor_SMD:C_0805_2012Metric
- C9: footprint (none) -> Capacitor_SMD:C_0805_2012Metric_Pad1.18x1.45mm_HandSolder
- F1: footprint (none) -> Fuse:Fuse_1206_3216Metric_Pad1.42x1.75mm_HandSolder
- J1: footprint (none) -> TerminalBlock_Phoenix:TerminalBlock_Phoenix_MKDS-1,5-2_1x02_P5.00mm_Horizontal
- J2: footprint (none) -> Connector_PinHeader_2.54mm:PinHeader_2x03_P2.54mm_Vertical
- J3, J4: footprint (none) -> Connector_Molex:Molex_KK-254_AE-6410-04A_1x04_P2.54mm_Vertical
- J5, J6, J7, J8: footprint (none) -> Connector_JST:JST_XH_B3B-XH-A_1x03_P2.50mm_Vertical
- J9: footprint (none) -> Connector_PinSocket_2.54mm:PinSocket_1x04_P2.54mm_Vertical
- R1, R10, R11, R2, R3, R4, R5, R6, R7, R8, R9: footprint (none) -> Resistor_SMD:R_0805_2012Metric
- SW1, SW2, SW3, SW4: footprint (none) -> Button_Switch_THT:SW_PUSH_6mm_H5mm
- Y1: footprint (none) -> Crystal:Crystal_HC49-U_Vertical
Other:
- note added: "FAN PWM"
- note added: "INTERFACE & MISC."
- note added: "MICROCONTROLLER"
- note added: "TEMP SENSORS"
- note added: "USB CABLE"
- moved on the sheet: C1, C10, C11, C2, C3, C4, C5, C6, C7, C8, C9, D1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

Commit message: PCB Complete
Other:
- moved on the sheet: R3, R5
Changed lines of the file:
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@@
 	)
 	(junction
-		(at 50.8 78.74)
+		(at 50.8 59.69)
 		(diameter 0)
 		(color 0 0 0 0)
@@
 	)
 	(junction
-		(at 50.8 59.69)
-		(diameter 0)
-		(color 0 0 0 0)
-	)
-	(junction
 		(at 152.4 76.2)
 		(diameter 0)
@@
 	)
 	(junction
+		(at 50.8 78.74)
+		(diameter 0)
+		(color 0 0 0 0)
+	)
+	(junction
 		(at 43.18 114.3)
 		(diameter 0)
@@
 	(wire
 		(pts
+			(xy 50.8 60.96) (xy 50.8 59.69)
+		)
+		(stroke
+			(width 0)
+			(type default)
+		)
+	)
+	(wire
+		(pts
 			(xy 54.61 78.74) (xy 50.8 78.74)
 		)
@@
 	(wire
 		(pts
+			(xy 50.8 80.01) (xy 50.8 78.74)
+		)
+		(stroke
+			(width 0)
+			(type default)
+		)
+	)
+	(wire
+		(pts
 			(xy 133.35 45.72) (xy 129.54 45.72)
 		)
@@
 	(symbol
 		(lib_id "Device:R")
-		(at 50.8 82.55 180)
+		(at 50.8 83.82 180)
 		(unit 1)
 		(body_style 1)
@@
 		(fields_autoplaced yes)
 		(property "Reference" "R5"
-			(at 53.34 81.2799 0)
+			(at 53.34 82.5499 0)
 			(show_name no)
 			(do_not_autoplace no)
@@
 		)
 		(property "Value" "10k"
-			(at 53.34 83.8199 0)
+			(at 53.34 85.0899 0)
 			(show_name no)
 			(do_not_autoplace no)
@@
 		)
 		(property "Footprint" "Resistor_SMD:R_0805_2012Metric"
-			(at 52.578 82.55 90)
+			(at 52.578 83.82 90)
 			(hide yes)
 			(show_name no)
@@
 		)
 		(property "Datasheet" ""
-			(at 50.8 82.55 0)
+			(at 50.8 83.82 0)
 			(hide yes)
 			(show_name no)
@@
 		)
 		(property "Description" "Resistor"
-			(at 50.8 82.55 0)
+			(at 50.8 83.82 0)
 			(hide yes)
 			(show_name no)
@@
 	(symbol
 		(lib_id "power:GND")
-		(at 50.8 86.36 0)
+		(at 50.8 87.63 0)
 		(unit 1)
 		(body_style 1)
@@
 		(fields_autoplaced yes)
 		(property "Reference" "#PWR020"
-			(at 50.8 92.71 0)
+			(at 50.8 93.98 0)
 			(hide yes)
 			(show_name no)
@@
 		)
 		(property "Value" "GND"
-			(at 50.8 91.44 0)
+			(at 50.8 92.71 0)
 			(show_name no)
 			(do_not_autoplace no)
@@
 		)
 		(property "Footprint" ""
-			(at 50.8 86.36 0)
+			(at 50.8 87.63 0)
 			(hide yes)
 			(show_name no)
@@
 		)
 		(property "Datasheet" ""
-			(at 50.8 86.36 0)
+			(at 50.8 87.63 0)
 			(hide yes)
 			(show_name no)
@@
 		)
 		(property "Description" "Power symbol creates a global label with name \"GND\" , ground"
-			(at 50.8 86.36 0)
+			(at 50.8 87.63 0)
 			(hide yes)
 			(show_name no)
@@
 	(symbol
 		(lib_id "Device:R")
-		(at 50.8 63.5 180)
+		(at 50.8 64.77 180)
 		(unit 1)
 		(body_style 1)
@@
 		(fields_autoplaced yes)
 		(property "Reference" "R3"
-			(at 53.34 62.2299 0)
+			(at 53.34 63.4999 0)
 			(show_name no)
 			(do_not_autoplace no)
@@
 		)
 		(property "Value" "10k"
-			(at 53.34 64.7699 0)
+			(at 53.34 66.0399 0)
 			(show_name no)
 			(do_not_autoplace no)
@@
 		)
 		(property "Footprint" "Resistor_SMD:R_0805_2012Metric"
-			(at 52.578 63.5 90)
+			(at 52.578 64.77 90)
 			(hide yes)
 			(show_name no)
@@
 		)
 		(property "Datasheet" ""
-			(at 50.8 63.5 0)
+			(at 50.8 64.77 0)
 			(hide yes)
 			(show_name no)
@@
 		)
 		(property "Description" "Resistor"
-			(at 50.8 63.5 0)
+			(at 50.8 64.77 0)
 			(hide yes)
 			(show_name no)
@@
 	(symbol
 		(lib_id "power:GND")
-		(at 50.8 67.31 0)
+		(at 50.8 68.58 0)
 		(unit 1)
 		(body_style 1)
@@
 		(fields_autoplaced yes)
 		(property "Reference" "#PWR019"
-			(at 50.8 73.66 0)
+			(at 50.8 74.93 0)
 			(hide yes)
 			(show_name no)
@@
 		)
 		(property "Value" "GND"
-			(at 50.8 72.39 0)
+			(at 50.8 73.66 0)
 			(show_name no)
 			(do_not_autoplace no)
@@
 		)
 		(property "Footprint" ""
-			(at 50.8 67.31 0)
+			(at 50.8 68.58 0)
 			(hide yes)
 			(show_name no)
@@
 		)
 		(property "Datasheet" ""
-			(at 50.8 67.31 0)
+			(at 50.8 68.58 0)
 			(hide yes)
 			(show_name no)
@@
 		)
 		(property "Description" "Power symbol creates a global label with name \"GND\" , ground"
-			(at 50.8 67.31 0)
+			(at 50.8 68.58 0)
 			(hide yes)
 			(show_name no)

Commit message: PCB Final
Parts:
- R10, R9: now not fitted
Changed lines of the file:
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@@
 		(on_board yes)
 		(in_pos_files yes)
-		(dnp no)
+		(dnp yes)
 		(property "Reference" "R9"
 			(at 194.3099 68.58 0)
@@
 		(on_board yes)
 		(in_pos_files yes)
-		(dnp no)
+		(dnp yes)
 		(property "Reference" "R10"
 			(at 204.4699 68.58 0)
